File: cap_water_sensor/cap_water_sensor.kicad_pcb (KiCad board)
At the start: 2 copper layers, 98 x 37.4 mm, 46 parts, among them P1 USB_C_Plug_USB2.0, SW2 SW_Push_Dual, U1 RP2040, U3 W25Q16JVSS, U5 MCP25625T-E/ML, Y1 AMB8G-12.0Hz

Commit message: changed sims and edits to pcb
Parts:
- added G***: LOGO, graphics:mamut, B.Cu at (189.2, 117.5)
- added G***: LOGO, graphics:gir, B.Cu at (193.8, 98.8)
- moved G 85.5 mm to (69.8, 111.0)
Routing:
- net unconnected-(R8-Pad1): track 0.00 -> 261.9 mm, vias 0 -> 1
- net (no net): track 0.00 -> 261.9 mm
- net +3V3: track 54.1 -> 62.1 mm, vias 1 -> 2
Other:
- board size 98 x 37.4 mm -> 136.6 x 37.5 mm
- board text added: "Health System :) By Sophia Garcia Version I 03/04"
