File: cap_water_sensor/cap_water_sensor.kicad_sch (KiCad schematic)
At the start: 45 parts, among them P1 USB_C_Plug_USB2.0, SW2 SW_Push_Dual, U1 RP2040, U3 W25Q16JVSS, U5 MCP25625T-E/ML, Y1 AMB8G-12.0Hz

Commit message: changed sims and edits to pcb
Changed lines of the file:
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@@
     (effects (font (size 1.27 1.27)) (justify left top))
   )
-  (text_box "Equation: C [capacitor] = A [area] x z [dielectric] / d [distance between plates]\nJCL dielectric for oridinary PCB product: z = 4.5 Farad/meter\nDistance between layers in JCL ordinary PBC product: d = 0.127 milimeters\nOptimized area for capacitor [length^{2} = A]: length = 3 centimeters\nFinal capacitor value: (0.03)^{2} x 4.5 / 0.127 x (10)^{-3} ~= 32 centifarad\n\n"
+  (text_box "Equation: C [capacitor] = A [area] x z [dielectric] / d [distance between plates]\nJCL dielectric for oridinary PCB product: z = 4.5 Farad/meter\nDistance between layers in JCL ordinary PBC product: d = 0.127 milimeters\nOptimized area for capacitor [length^{2} = A]: length = 1 milimeters\nFinal capacitor value: (0.001)^{2} x 4.5 / 0.127 x (10)^{-3} ~= 3.5 centifarad\n\n"
     (at 15.24 15.24 0) (size 68.58 19.05)
     (stroke (width 0) (type default))
